File: hps-schematic-2.0.kicad_sch (KiCad schematic)
At the start: 50 parts, among them J1 Conn_02x03_Odd_Even, J1(POWER)1 PJ-102AH, J2 Conn_01x06, U2(POWER)1 L7805, Y1 Crystal_32768Hz

Commit message: Schematic/PCB Update
Parts:
- J1(POWER)1: footprint footprints:PJ-102AH -> footprints:Wurth-694106402002; symbol HPS:PJ-102AH -> HPS:Power_inlet_vertical; Digikey PN CP-102AH-ND -> 732-5931-ND; MFG CUI Devices -> Wurth; MPN PJ-102AH -> 694106402002
Changed lines of the file:
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@@
     (pin "6")
   )
-  (symbol (lib_id "HPS:PJ-102AH") (at 156.21 29.21 0) (unit 1)
-    (in_bom yes) (on_board yes) (fields_autoplaced)
+  (symbol (lib_id "HPS:Power_inlet_vertical") (at 156.21 29.21 0) (unit 1)
+    (in_bom yes) (on_board yes)
     (property "Reference" "J1(POWER)1" (id 0) (at 153.67 16.51 0)
       (effects (font (size 1.524 1.524)))
@@
       (effects (font (size 1.524 1.524)))
     )
-    (property "Footprint" "footprints:PJ-102AH" (id 2) (at 153.67 24.13 0)
+    (property "Footprint" "footprints:Wurth-694106402002" (id 2) (at 143.51 34.29 90)
       (effects (font (size 1.524 1.524)))
     )
-    (property "Datasheet" "https://www.cuidevices.com/product/resource/pj-102ah.pdf" (id 3) (at 157.734 41.148 0)
+    (property "Datasheet" "https://www.we-online.com/katalog/datasheet/6941xx402002.pdf" (id 3) (at 157.734 41.148 0)
       (effects (font (size 1.524 1.524)) hide)
     )
-    (property "MFG" "CUI Devices" (id 4) (at 156.21 46.99 0)
-      (effects (font (size 1.27 1.27)) hide)
-    )
-    (property "MPN" "PJ-102AH" (id 5) (at 156.21 49.53 0)
-      (effects (font (size 1.27 1.27)) hide)
-    )
-    (property "Digikey PN" "CP-102AH-ND" (id 6) (at 157.734 54.737 0)
+    (property "MFG" "Wurth" (id 4) (at 156.21 46.99 0)
+      (effects (font (size 1.27 1.27)) hide)
+    )
+    (property "MPN" "694106402002" (id 5) (at 156.21 49.53 0)
+      (effects (font (size 1.27 1.27)) hide)
+    )
+    (property "Digikey PN" "732-5931-ND" (id 6) (at 157.734 54.737 0)
       (effects (font (size 1.27 1.27)) hide)
     )
@@
     )
     (path "/0dbb3083-2dbf-40a3-82c6-9cc694e803d7"
-      (reference "J1(POWER)1") (unit 1) (value "PJ-102AH") (footprint "footprints:PJ-102AH")
+      (reference "J1(POWER)1") (unit 1) (value "PJ-102AH") (footprint "footprints:Wurth-694106402002")
     )
     (path "/d2e60283-9e54-4f91-bab9-eea8b7c8a850"

Commit message: Schematic/PCB Update
Connections:
- no-connect marks 10 -> 14
Changed lines of the file:
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@@
   (no_connect (at 74.93 55.88))
   (no_connect (at 74.93 81.28))
+  (no_connect (at 175.26 146.05))
+  (no_connect (at 175.26 148.59))
+  (no_connect (at 175.26 151.13))
+  (no_connect (at 175.26 153.67))
   (wire (pts (xy 43.18 166.37) (xy 41.91 166.37))
     (stroke (width 0) (type default) (color 0 0 0 0))

Commit message: Gerber Out
Changed lines of the file:
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@@
     (pin "1")
   )
-  (symbol (lib_id "HPS:MountingHole") (at 45.72 179.07 0) (unit 1)
+  (symbol (lib_name "MountingHole_3") (lib_id "HPS:MountingHole") (at 45.72 179.07 0) (unit 1)
     (in_bom yes) (on_board yes) (fields_autoplaced)
     (property "Reference" "H3" (id 0) (at 48.26 177.7999 0)
@@
     (pin "2")
   )
-  (symbol (lib_id "HPS:MountingHole") (at 25.4 179.07 0) (unit 1)
+  (symbol (lib_name "MountingHole_1") (lib_id "HPS:MountingHole") (at 25.4 179.07 0) (unit 1)
     (in_bom yes) (on_board yes) (fields_autoplaced)
     (property "Reference" "H1" (id 0) (at 27.94 177.7999 0)
@@
     (pin "1")
   )
-  (symbol (lib_id "HPS:MountingHole") (at 25.4 186.69 0) (unit 1)
+  (symbol (lib_name "MountingHole_2") (lib_id "HPS:MountingHole") (at 25.4 186.69 0) (unit 1)
     (in_bom yes) (on_board yes) (fields_autoplaced)
     (property "Reference" "H2" (id 0) (at 27.94 185.4199 0)
