File: hps-schematic-2.0.kicad_pcb (KiCad board)
At the start: 2 copper layers, 140 x 90 mm, 50 parts, among them J1 Conn_02x03_Odd_Even, J1(POWER)1 PJ-102AH, J2 Conn_01x06, U2(POWER)1 L7805, Y1 Crystal_32768Hz

Commit message: Schematic/PCB Update
Parts:
- J1(POWER)1: footprint footprints:PJ-102AH -> footprints:Wurth-694106402002
- moved TP1 95.1 mm to (86.4, 78.7)
- moved TP2 71.3 mm to (83.8, 109.2)
- moved TP9 47.8 mm to (179.3, 118.4)
- moved TP10 47.0 mm to (106.7, 124.5)
- moved TP8 45.0 mm to (177.8, 132.1)
- moved TP4 45.0 mm to (132.1, 119.4)
- moved TP3 37.1 mm to (137.2, 119.4)
- moved TP6 34.2 mm to (144.8, 119.4)
- moved TP7 29.8 mm to (160.0, 139.7)
- moved TP5 24.8 mm to (165.1, 139.7)
- moved TP11 18.1 mm to (147.3, 139.7)
Routing:
- net VCC: track 23.4 -> 69.4 mm
- net MATRIX_DIN: track 109.4 -> 118.8 mm
- net MATRIX_CLK: track 79.6 -> 89.0 mm
- net GND: track 79.9 -> 84.8 mm, vias 24 -> 26
- net SCL: track 20.6 -> 25.0 mm
- net SDA: track 18.8 -> 23.2 mm
- net Net-(C6-Pad1): track 39.4 -> 35.8 mm
- net MATRIX_CS: track 68.4 -> 70.9 mm

Commit message: Schematic/PCB Update
Routing:
- net VCC: track 69.4 -> 83.0 mm, vias 0 -> 3
- net SCL: vias 2 -> 1
Changed lines of the file:
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@@
     (property "Tolerance" "N/A")
     (attr smd)
-    (fp_text reference "R6" (at 0 -1.65 90) (layer "F.SilkS")
+    (fp_text reference "R6" (at 2.54 0 180) (layer "F.SilkS")
       (effects (font (size 1 1) (thickness 0.15)))
     )
@@
     (property "Tolerance" "N/A")
     (attr smd)
-    (fp_text reference "R7" (at 0 -1.65 90) (layer "F.SilkS")
+    (fp_text reference "R7" (at 2.54 0 180) (layer "F.SilkS")
       (effects (font (size 1 1) (thickness 0.15)))
     )
@@
     (property "Tolerance" "N/A")
     (attr smd)
-    (fp_text reference "R4" (at 0 -1.65) (layer "F.SilkS")
+    (fp_text reference "R4" (at 0 2.54) (layer "F.SilkS")
       (effects (font (size 1 1) (thickness 0.15)))
     )
@@
     (property "Voltage" "N/A")
     (attr smd)
-    (fp_text reference "C5" (at 0 -1.65 90) (layer "F.SilkS")
+    (fp_text reference "C5" (at 2.54 0 180) (layer "F.SilkS")
       (effects (font (size 1 1) (thickness 0.15)))
     )
@@
     (property "Sheetname" "")
     (attr exclude_from_pos_files)
-    (fp_text reference "TP7" (at 0 -1.998) (layer "F.SilkS")
+    (fp_text reference "TP7" (at 0 2.54) (layer "F.SilkS")
       (effects (font (size 1 1) (thickness 0.15)))
     )
@@
       (effects (font (size 1 1) (thickness 0.15)) (justify right))
     )
-    (fp_text value "LED_Display_1001" (at 0 0 90) (layer "F.SilkS")
+    (fp_text value "LED_Display_1001" (at -12.7 -20.32 180) (layer "F.SilkS")
       (effects (font (size 1.27 1.27) (thickness 0.15)))
     )
@@
     (property "Voltage" "N/A")
     (attr smd)
-    (fp_text reference "C6" (at 0 -1.65) (layer "F.SilkS")
+    (fp_text reference "C6" (at -2.54 0) (layer "F.SilkS")
       (effects (font (size 1 1) (thickness 0.15)))
     )
@@
     (property "Voltage" "N/A")
     (attr smd)
-    (fp_text reference "C2" (at 0 -1.65 90) (layer "F.SilkS")
+    (fp_text reference "C2" (at -2.54 2.54 180) (layer "F.SilkS")
       (effects (font (size 1 1) (thickness 0.15)))
     )
@@
     (property "Sheetname" "")
     (attr smd)
-    (fp_text reference "CRYSTAL1" (at 0 -3.55) (layer "F.SilkS")
+    (fp_text reference "CRYSTAL1" (at -0.4 5.08) (layer "F.SilkS")
       (effects (font (size 1 1) (thickness 0.15)))
     )
@@
     (property "Sheetname" "")
     (attr exclude_from_pos_files)
-    (fp_text reference "TP11" (at 0 -1.998) (layer "F.SilkS")
+    (fp_text reference "TP11" (at 0 2.54) (layer "F.SilkS")
       (effects (font (size 1 1) (thickness 0.15)))
     )
@@
     (property "Sheetname" "")
     (attr through_hole)
-    (fp_text reference "J1(POWER)1" (at 0 5 90 unlocked) (layer "B.SilkS")
+    (fp_text reference "J1(POWER)1" (at 7.62 -7.62 unlocked) (layer "B.SilkS")
       (effects (font (size 1 1) (thickness 0.15)) (justify mirror))
     )
@@
   (segment (start 91.44 92.705) (end 90.175 92.705) (width 0.2032) (layer "F.Cu") (net 2))
   (segment (start 149.86 121.92) (end 148.6 123.18) (width 0.2032) (layer "F.Cu") (net 2))
+  (segment (start 187.79 99.06) (end 180.34 99.06) (width 0.2032) (layer "F.Cu") (net 2))
   (segment (start 144.76 137.14) (end 144.78 137.16) (width 0.2032) (layer "F.Cu") (net 2))
   (segment (start 204.05 137.16) (end 205.74 137.16) (width 0.2032) (layer "F.Cu") (net 2))
@@
   (segment (start 140.55 135.47) (end 139.7 134.62) (width 0.2032) (layer "F.Cu") (net 2))
   (segment (start 92.25 120.905) (end 93.775 119.38) (width 0.2032) (layer "F.Cu") (net 2))
+  (via (at 180.34 99.06) (size 0.8128) (drill 0.4064) (layers "F.Cu" "B.Cu") (net 2))
   (via (at 83.82 104.14) (size 0.8128) (drill 0.4064) (layers "F.Cu" "B.Cu") (net 2))
   (via (at 134.62 68.58) (size 0.8128) (drill 0.4064) (layers "F.Cu" "B.Cu") (net 2))
@@
   (via (at 106.68 127) (size 0.8128) (drill 0.4064) (layers "F.Cu" "B.Cu") (net 2))
   (via (at 205.74 137.16) (size 0.8128) (drill 0.4064) (layers "F.Cu" "B.Cu") (net 2))
-  (via (at 180.34 99.06) (size 0.8128) (drill 0.4064) (layers "F.Cu" "B.Cu") (net 2))
   (via (at 175.26 68.58) (size 0.8128) (drill 0.4064) (layers "F.Cu" "B.Cu") (net 2))
-  (segment (start 187.79 99.06) (end 180.34 99.06) (width 0.2032) (layer "B.Cu") (net 2))
   (segment (start 144.105689 131.904311) (end 147.495689 131.904311) (width 0.2032) (layer "F.Cu") (net 3))
+  (segment (start 106.68 99.06) (end 101.6 99.06) (width 0.2032) (layer "F.Cu") (net 3))
   (segment (start 142.24 133.77) (end 144.105689 131.904311) (width 0.2032) (layer "F.Cu") (net 3))
+  (segment (start 105.83 102.45) (end 106.68 101.6) (width 0.2032) (layer "F.Cu") (net 3))
   (segment (start 120.22 120.22) (end 118.12 118.12) (width 0.2032) (layer "F.Cu") (net 3))
   (segment (start 147.495689 131.904311) (end 148.6 130.8) (width 0.2032) (layer "F.Cu") (net 3))
@@
   (segment (start 124.46 123.61) (end 124.46 119.38) (width 0.2032) (layer "F.Cu") (net 3))
   (segment (start 124.46 119.38) (end 123.2 118.12) (width 0.2032) (layer "F.Cu") (net 3))
+  (segment (start 104.14 102.45) (end 105.83 102.45) (width 0.2032) (layer "F.Cu") (net 3))
+  (via (at 106.68 99.06) (size 0.8128) (drill 0.4064) (layers "F.Cu" "B.Cu") (net 3))
+  (via (at 106.68 101.6) (size 0.8128) (drill 0.4064) (layers "F.Cu" "B.Cu") (net 3))
+  (via (at 101.6 99.06) (size 0.8128) (drill 0.4064) (layers "F.Cu" "B.Cu") (net 3))
   (segment (start 83.82 109.22) (end 83.82 106.383267) (width 0.2032) (layer "B.Cu") (net 3))
   (segment (start 91.313956 98.889311) (end 97.955689 98.889311) (width 0.2032) (layer "B.Cu") (net 3))
@@
   (segment (start 106.68 122.918267) (end 110.373956 119.224311) (width 0.2032) (layer "B.Cu") (net 3))
   (segment (start 110.373956 119.224311) (end 117.015689 119.224311) (width 0.2032) (layer "B.Cu") (net 3))
+  (segment (start 99.06 97.785) (end 100.325 97.785) (width 0.2032) (layer "B.Cu") (net 3))
   (segment (start 147.32 132.08) (end 148.6 130.8) (width 0.2032) (layer "B.Cu") (net 3))
+  (segment (start 100.325 97.785) (end 101.6 99.06) (width 0.2032) (layer "B.Cu") (net 3))
   (segment (start 147.32 139.7) (end 147.32 132.08) (width 0.2032) (layer "B.Cu") (net 3))
   (segment (start 97.955689 98.889311) (end 99.06 97.785) (width 0.2032) (layer "B.Cu") (net 3))
+  (segment (start 106.68 101.6) (end 106.68 99.06) (width 0.2032) (layer "B.Cu") (net 3))
   (segment (start 106.68 124.46) (end 106.68 122.918267) (width 0.2032) (layer "B.Cu") (net 3))
   (segment (start 83.82 106.383267) (end 91.313956 98.889311) (width 0.2032) (layer "B.Cu") (net 3))
@@
   (segment (start 119.4 121.92) (end 118.12 123.2) (width 0.2032) (layer "F.Cu") (net 23))
   (segment (start 121.92 121.92) (end 119.4 121.92) (width 0.2032) (layer "F.Cu") (net 23))
-  (via (at 121.92 121.92) (size 0.8128) (drill 0.4064) (layers "F.Cu" "B.Cu") (net 23))
   (via (at 127 121.92) (size 0.8128) (drill 0.4064) (layers "F.Cu" "B.Cu") (net 23))
   (segment (start 127 121.92) (end 125.72 123.2) (width 0.2032) (layer "B.Cu") (net 23))
@@
   (via (at 109.22 132.08) (size 0.8128) (drill 0.4064) (layers "F.Cu" "B.Cu") (net 37))
   (segment (start 109.22 132.08) (end 109.22 124.48) (width 0.2032) (layer "B.Cu") (net 37))
-  (segment (start 109.22 124.48) (end 109.2 124.46) (width 0.2032) (layer "B.Cu") (net 37))
   (segment (start 182.88 127) (end 208.28 101.6) (width 0.2032) (layer "B.Cu") (net 37))
   (segment (start 109.22 124.48) (end 110.5 123.2) (width 0.2032) (layer "B.Cu") (net 37))
@@
   (segment (start 106.68 106.68) (end 104.14 104.14) (width 0.2032) (layer "F.Cu") (net 40))
   (via (at 104.14 104.14) (size 0.8128) (drill 0.4064) (layers "F.Cu" "B.Cu") (net 40))
-  (segment (start 104.14 104.14) (end 104.14 95.245) (width 0.2032) (layer "B.Cu") (net 40))
-  (segment (start 104.14 95.245) (end 99.06 90.165) (width 0.2032) (layer "B.Cu") (net 40))
+  (segment (start 99.06 90.165) (end 104.14 95.245) (width 0.2032) (layer "B.Cu") (net 40))
+  (segment (start 104.14 95.245) (end 104.14 104.14) (width 0.2032) (layer "B.Cu") (net 40))
   (segment (start 113.035 95.245) (end 99.06 95.245) (width 0.2032) (layer "F.Cu") (net 41))
   (segment (start 149.86 91.44) (end 147.32 88.9) (width 0.2032) (layer "F.Cu") (net 41))
@@
   (segment (start 147.32 91.44) (end 135.330701 103.429299) (width 0.2032) (layer "F.Cu") (net 42))
   (segment (start 135.330701 103.429299) (end 99.624299 103.429299) (width 0.2032) (layer "F.Cu") (net 42))
-  (segment (start 144.78 92.445084) (end 138.004395 99.220689) (width 0.2032) (layer "F.Cu") (net 43))
+  (segment (start 137.454383 99.770701) (end 101.176032 99.770701) (width 0.2032) (layer "F.Cu") (net 43))
   (segment (start 92.544311 101.429311) (end 91.44 100.325) (width 0.2032) (layer "F.Cu") (net 43))
-  (segment (start 138.004395 99.220689) (end 101.726044 99.220689) (width 0.2032) (layer "F.Cu") (net 43))
+  (segment (start 144.78 92.445084) (end 137.454383 99.770701) (width 0.2032) (layer "F.Cu") (net 43))
+  (segment (start 101.176032 99.770701) (end 99.517422 101.429311) (width 0.2032) (layer "F.Cu") (net 43))
   (segment (start 99.517422 101.429311) (end 92.544311 101.429311) (width 0.2032) (layer "F.Cu") (net 43))
-  (segment (start 101.726044 99.220689) (end 99.517422 101.429311) (width 0.2032) (layer "F.Cu") (net 43))
   (segment (start 144.78 91.44) (end 144.78 92.445084) (width 0.2032) (layer "F.Cu") (net 43))
   (segment (start 142.24 91.44) (end 98.773267 91.44) (width 0.2032) (layer "F.Cu") (net 44))
@@
   )
   (zone locked (net 3) (net_name "VCC") (layer "F.Cu") (hatch edge 0.508)
-    (connect_pads (clearance 0))
-    (min_thickness 0.254) (filled_areas_thickness no)
+    (connect_pads (clearance 0.3048))
+    (min_thickness 0.3048) (filled_areas_thickness no)
     (fill yes (thermal_gap 0.3048) (thermal_bridge_width 0.508))
     (polygon
@@
   )
   (zone (net 2) (net_name "GND") (layer "B.Cu") (hatch edge 0.508)
-    (connect_pads (clearance 0))
-    (min_thickness 0.254) (filled_areas_thickness no)
+    (connect_pads (clearance 0.3048))
+    (min_thickness 0.3048) (filled_areas_thickness no)
     (fill yes (thermal_gap 0.3048) (thermal_bridge_width 0.508))
     (polygon

Commit message: Gerber Out
Other:
- board text added: "LIL BEN"

Commit message: Gerber Out 2.0
Parts:
- moved J1(POWER)1 8.89 mm to (97.8, 129.5)
- turned DS1 to 90 degrees
Routing:
- net Net-(DS1-Pad7): track 51.3 -> 101.5 mm, vias 0 -> 2
- net Net-(DS1-Pad14): track 99.5 -> 68.2 mm
- net Net-(DS1-Pad9): track 48.0 -> 74.5 mm, vias 0 -> 1
- net Net-(DS1-Pad11): track 64.0 -> 80.3 mm
- net Net-(DS1-Pad6): track 58.5 -> 70.8 mm, vias 0 -> 1
- net Net-(DS1-Pad3): track 74.7 -> 85.2 mm, vias 1 -> 3
- net Net-(DS1-Pad12): track 70.9 -> 80.3 mm
- net Net-(C6-Pad1): track 35.8 -> 44.7 mm
- net Net-(DS1-Pad13): track 57.5 -> 65.6 mm, vias 0 -> 2
- net Net-(DS1-Pad2): track 57.5 -> 65.6 mm, vias 0 -> 1
- net Net-(DS1-Pad4): track 57.5 -> 62.2 mm, vias 2 -> 3
- net Net-(DS1-Pad5): track 53.5 -> 57.5 mm, vias 0 -> 1
- net Net-(DS1-Pad10): track 67.2 -> 65.1 mm
- net Net-(DS1-Pad1): track 76.7 -> 76.0 mm
